Commit message: boao v1

File: src/publish_ship_model/try.urdf (robot description, URDF)
Before this commit: robot example_robot, 2 links, 1 joints
Links:
- removed link hesai_at128
- added link ship_center; visual cylinder length=0.5 radius=0.1
Joints:
- joint base_to_lidar: child hesai_at128 -> ship_center
